Commit message: updated boat model

File: CSEI/boat_model/urdf/boat.urdf (robot description, URDF)
Before this commit: robot myfirst, 1 links, 0 joints
Links:
- link base_link: geometry visual mesh filename=package://boat_model/meshes/lowpolyship.stl scale=0.018 0.018 0.018

Commit message: update

File: CSEI/boat_model/urdf/boat.urdf (robot description, URDF)
Before this commit: robot myfirst, 1 links, 0 joints
Links:
- link base_link: geometry visual mesh filename=package://boat_model/meshes/lowpolyship.stl scale=0.010 0.010 0.010
